Commit message: Upgrade the gazebo9

File: ur_description/urdf/common.gazebo.xacro (robot description, xacro)
@@ -22,3 +22,51 @@
 -->
   </gazebo>
+  <material name="Blue">
+      <color rgba="0.0 0.0 0.8 1.0"/>
+    </material>
+    <material name="Green">
+      <color rgba="0.0 0.8 0.0 1.0"/>
+    </material>
+    <material name="Grey">
+      <color rgba="0.7 0.7 0.7 1.0"/>
+    </material>
+    <material name="LightGrey">
+      <color rgba="0.95 0.95 0.95 1.0"/>
+    </material>
+    <material name="DarkGrey">
+      <color rgba="0.1 0.1 0.1 1.0"/>
+    </material>
+    <material name="Red">
+      <color rgba="0.8 0.0 0.0 1.0"/>
+    </material>
+    <material name="White">
+      <color rgba="1.0 1.0 1.0 1.0"/>
+    </material>
+    <material name="Yellow">
+      <color rgba="0.96 0.88 0.14 1.0"/>
+    </material>
+  <gazebo reference="base_link">
+    <material>Gazebo/LightGrey</material>
+  </gazebo>
+  <gazebo reference="shoulder_link">
+    <material>Gazebo/LightGrey</material>
+  </gazebo>
+  <gazebo reference="upper_arm_link">
+    <material>Gazebo/LightGrey</material>
+  </gazebo>
+  <gazebo reference="forearm_link">
+    <material>Gazebo/LightGrey</material>
+  </gazebo>
+  <gazebo reference="wrist_1_link">
+    <material>Gazebo/LightGrey</material>
+  </gazebo>
+  <gazebo reference="wrist_2_link">
+    <material>Gazebo/LightGrey</material>
+  </gazebo>
+  <gazebo reference="wrist_3_link">
+    <material>Gazebo/LightGrey</material>
+  </gazebo>
+  <gazebo reference="ee_link">
+    <material>Gazebo/LightGrey</material>
+  </gazebo>
 </robot>

Commit message: Find the gazebo segmentation error

File: ur_description/urdf/common.gazebo.xacro (robot description, xacro)
@@ -70,3 +70,30 @@
     <material>Gazebo/LightGrey</material>
   </gazebo>
+  <gazebo>
+    <plugin name="camera_plugin" filename="libgazebo_ros_openni_kinect.so">
+      <baseline>0.2</baseline>
+      <alwaysOn>true</alwaysOn>
+      <!-- Keep this zero, update_rate in the parent <sensor> tag
+        will control the frame rate. -->
+      <updateRate>0.0</updateRate>
+      <cameraName>camera_ir</cameraName>
+      <imageTopicName>/camera/depth/image_raw</imageTopicName>
+      <cameraInfoTopicName>/camera/depth/camera_info</cameraInfoTopicName>
+      <depthImageTopicName>/camera/depth/image_raw</depthImageTopicName>
+      <depthImageInfoTopicName>/camera/depth/camera_info</depthImageInfoTopicName>
+      <pointCloudTopicName>/camera/depth/points</pointCloudTopicName>
+      <frameName>camera_link</frameName>
+      <pointCloudCutoff>0.05</pointCloudCutoff>
+      <distortionK1>0</distortionK1>
+      <distortionK2>0</distortionK2>
+      <distortionK3>0</distortionK3>
+      <distortionT1>0</distortionT1>
+      <distortionT2>0</distortionT2>
+      <CxPrime>0</CxPrime>
+      <Cx>0</Cx>
+      <Cy>0</Cy>
+      <focalLength>0</focalLength>
+      <hackBaseline>0</hackBaseline>
+    </plugin>
+  </gazebo>
 </robot>

File: ur_description/urdf/hand.urdf.xacro (robot description, xacro)
@@ -1,4 +1,4 @@
 <?xml version="1.0" encoding="utf-8"?>
-<robot xmlns:xacro="http://www.ros.org/wiki/xacro" name="hand">
+<robot xmlns:xacro="http://wiki.ros.org/xacro" name="hand">
   <xacro:include filename="hand.xacro"/>
   <xacro:hand ns="ur5"/>

File: ur_description/urdf/hand.xacro (robot description, xacro)
@@ -1,4 +1,4 @@
 <?xml version="1.0" encoding="utf-8"?>
-<robot xmlns:xacro="http://www.ros.org/wiki/xacro" name="hand">
+<robot xmlns:xacro="http://wiki.ros.org/xacro" name="hand">
   <xacro:macro name="hand" params="connected_to:='' ns:='' rpy:='0 0 0' xyz:='0 0 0' ">
     <xacro:unless value="${connected_to == ''}">
@@ -12,10 +12,10 @@
       <visual>
         <geometry>
-          <mesh filename="package://franka_description/meshes/visual/hand.dae"/>
+          <mesh filename="package://ur_description/meshes/hand/visual/hand.dae"/>
         </geometry>
       </visual>
       <collision>
         <geometry>
-          <mesh filename="package://franka_description/meshes/collision/hand.stl"/>
+          <mesh filename="package://ur_description/meshes/hand/collision/hand.stl"/>
         </geometry>
       </collision>
@@ -24,10 +24,10 @@
       <visual>
         <geometry>
-          <mesh filename="package://franka_description/meshes/visual/finger.dae"/>
+          <mesh filename="package://ur_description/meshes/hand/visual/finger.dae"/>
         </geometry>
       </visual>
       <collision>
         <geometry>
-          <mesh filename="package://franka_description/meshes/collision/finger.stl"/>
+          <mesh filename="package://ur_description/meshes/hand/collision/finger.stl"/>
         </geometry>
       </collision>
@@ -37,5 +37,5 @@
         <origin xyz="0 0 0" rpy="0 0 ${pi}"/>
         <geometry>
-          <mesh filename="package://franka_description/meshes/visual/finger.dae"/>
+          <mesh filename="package://ur_description/meshes/hand/visual/finger.dae"/>
         </geometry>
       </visual>
@@ -43,5 +43,5 @@
         <origin xyz="0 0 0" rpy="0 0 ${pi}"/>
         <geometry>
-          <mesh filename="package://franka_description/meshes/collision/finger.stl"/>
+          <mesh filename="package://ur_description/meshes/hand/collision/finger.stl"/>
         </geometry>
       </collision>

File: ur_description/urdf/ur.gazebo.xacro (robot description, xacro)
@@ -1,4 +1,4 @@
 <?xml version="1.0"?>
-<robot xmlns:xacro="http://wiki.ros.org/xacro">
+<robot  name="ur5" xmlns:xacro="http://ros.org/wiki/xacro" >
   <xacro:macro name="ur_arm_gazebo" params="prefix">
     <gazebo reference="${prefix}shoulder_link">

File: ur_description/urdf/ur.transmission.xacro (robot description, xacro)
@@ -1,4 +1,4 @@
 <?xml version="1.0"?>
-<robot xmlns:xacro="http://wiki.ros.org/xacro">
+<robot xmlns:xacro="http://wiki.ros.org/xacro" name="ur5">
   <xacro:macro name="ur_arm_transmission" params="prefix">
     <transmission name="${prefix}shoulder_pan_trans">

File: ur_description/urdf/ur5.urdf.xacro (robot description, xacro)
@@ -1,4 +1,4 @@
 <?xml version="1.0"?>
-<robot xmlns:xacro="http://wiki.ros.org/xacro">
+<robot name="ur5" xmlns:xacro="http://ros.org/wiki/xacro">
   <xacro:include filename="$(find ur_description)/urdf/ur.transmission.xacro" />
   <xacro:include filename="$(find ur_description)/urdf/ur.gazebo.xacro" />

File: ur_description/urdf/ur5_hand.urdf.xacro (robot description, xacro)
@@ -1,4 +1,4 @@
 <?xml version="1.0" ?>
-<robot xmlns:xacro="http://www.ros.org/wiki/xacro" name="ur5">
+<robot  name="ur5" xmlns:xacro="http://ros.org/wiki/xacro">
   <!-- common stuff -->
   <xacro:include filename="$(find ur_description)/urdf/common.gazebo.xacro" />
@@ -6,9 +6,10 @@
   <xacro:include filename="$(find ur_description)/urdf/ur5.urdf.xacro" />
   <!-- hand -->
-  <xacro:include filename="$(find franka_description)/robots/hand.xacro"/>
+  <xacro:include filename="$(find ur_description)/urdf/hand.xacro"/>
   <!-- arm -->
   <xacro:ur5_robot prefix="" joint_limited="false"/>
   <xacro:hand ns="ur5" rpy="0 ${pi/2} 0" connected_to="ee_link"/>
-  <link name="world" />
+  <link name="world" >
+  </link>
   <joint name="world_joint" type="fixed">
     <parent link="world" />
@@ -16,3 +17,15 @@
     <origin xyz="0.0 0.0 0.60" rpy="0.0 0.0 0.0" />
   </joint>
+  <link name="camera_rgb_optical_frame">
+    <visual>
+      <geometry>
+      <mesh filename="package://ur_description/meshes/kinect/meshes/kinect.dae"/>
+      </geometry>
+    </visual>
+  </link>
+  <joint name="camera_joint" type="fixed">
+    <parent link="world" />
+    <child link = "camera_rgb_optical_frame" />
+    <origin xyz="0.0 0.0 2.0" rpy="0.0 ${pi/2} 0.0" />
+  </joint>
 </robot>

File: ur_description/urdf/ur5_robot.urdf.xacro (robot description, xacro)
@@ -1,5 +1,4 @@
 <?xml version="1.0"?>
-<robot xmlns:xacro="http://wiki.ros.org/xacro"
-       name="ur5" >
+<robot name="ur5" xmlns:xacro="http://ros.org/wiki/xacro">
   <!-- common stuff -->
   <xacro:include filename="$(find ur_description)/urdf/common.gazebo.xacro" />
