Commit message: Replace new grip_moveit

File: ur_description/urdf/ur5_hand.urdf.xacro (robot description, xacro)
@@ -10,3 +10,9 @@
   <xacro:ur5_robot prefix="" joint_limited="false"/>
   <xacro:hand ns="ur5" rpy="0 ${pi/2} 0" connected_to="ee_link"/>
+  <link name="world" />
+  <joint name="world_joint" type="fixed">
+    <parent link="world" />
+    <child link = "base_link" />
+    <origin xyz="0.0 0.0 0.60" rpy="0.0 0.0 0.0" />
+  </joint>
 </robot>

Commit message: ur5 moveit exection

File: ur_description/urdf/ur5_hand.urdf.xacro (robot description, xacro)
@@ -15,5 +15,5 @@
     <parent link="world" />
     <child link = "base_link" />
-    <origin xyz="0.0 0.0 0.60" rpy="0.0 0.0 0.0" />
+    <origin xyz="0.0 0.0 1.00" rpy="0.0 0.0 0.0" />
   </joint>
   <link name="camera_rgb_optical_frame">
